File: hardware/exopet-hat/exopet-hat.kicad_pcb (KiCad board)
At the start: 2 copper layers, 65 x 56 mm, 71 parts, among them J1 BarrelJack_CUI_PJ-102AH_Horiz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, J10 TerminalBlock_Phoenix_PT-1,5-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, J11 TerminalBlock_Phoenix_PT-1,5-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, J13 TerminalBlock_Phoenix_PT-1,5-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, J14 TerminalBlock_Phoenix_PT-1,5-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, J3 PinSocket_2x20_P2.54mm_Vertic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, J4 TerminalBlock_Phoenix_PT-1,5-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, J8 TerminalBlock_Phoenix_PT-1,5-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, J9 TerminalBlock_Phoenix_PT-1,5-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, K1 Relay_SPDT_Omron-G5LE-1, K2 Relay_SPDT_Omron-G5LE-1, K3 Relay_SPDT_Omron-G5LE-1, K4 Relay_SPDT_Omron-G5LE-1, Q1 TO-252-2, U2 SOIC-16_3.9x9.9mm_P1.27mm, U4 SOIC-8_3.9x4.9mm_P1.27mm, U5 D_SOD-323, U6 SOT-23-6

Commit message: HAT: fix netless Q1 — root cause of rev 1's dead relays
Device:Q_PMOS uses letters (D/G/S) as pin numbers while the TO-252
footprint pads are 1/2/3; gen_board's net lookup silently missed, so
Q1 shipped with NO nets on rev 1: the +12V rail (all relay coils) was
an island with no source. Bench symptom: GPIO toggles perfectly,
relays never click, regardless of D1.

Fix: PAD_PIN_MAP (pad1=G, pad2=D/tab, pad3=S per AOD403) + a build
guard asserting every netlist pin lands on a footprint pad. Q1 added
to the polarity lint. Rev 2 rerouted: DRC 0/0, renders + gerbers
refreshed. Rev 1 bench workaround: jumper F1-out to PSU1 VIN (bypasses
the never-functional Q1) after confirming a center-positive supply.

Co-Authored-By: Claude Fable 5 <noreply@anthropic.com>
Connections:
- Q1 pad 1: (no net) -> Q1_G
- Q1 pad 2: (no net) -> +12V_F
- Q1 pad 3: (no net) -> +12V
Routing:
- net CH2_OUT: track 122.1 -> 61.2 mm, vias 0 -> 1
- net CH1_FUSED: track 81.7 -> 31.3 mm, vias 0 -> 1
- net RLY4_DRV: track 97.8 -> 68.2 mm, vias 0 -> 1
- net LED1_A: track 87.3 -> 62.1 mm, vias 1 -> 3
- net +12V_F: track 44.3 -> 68.7 mm
- net +12V: track 167.4 -> 189.4 mm
- net +3V3: track 153.3 -> 175.2 mm, vias 0 -> 2
- net +5V_BUCK: track 79.6 -> 58.7 mm, vias 2 -> 3
- net BUCK_FB: track 58.5 -> 40.3 mm
- net CH1_OUT: track 98.5 -> 116.2 mm, vias 1 -> 0
- net LED2_A: track 67.9 -> 50.5 mm
- net GND: track 306.0 -> 290.9 mm, vias 0 -> 1
- net RLY2_DRV: track 84.0 -> 96.9 mm
- net +5V: track 87.2 -> 74.5 mm
- net RLY3_DRV: track 46.2 -> 56.6 mm
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
Commit message: HAT rev 2: deep-QA suite — golden audit, fab cross-check, preflight gate
check_golden.py: hand-written design-intent table (67 parts, 208 pins)
verified against BOTH the netlist and the routed board's copper —
independent of the generators, so shared-assumption bugs (netless Q1,
backwards D1) cannot pass. Includes full-coverage sweep: no pad on the
board escapes the audit. check_fab.py cross-checks BOM/CPL against the
board. preflight.sh regenerates and runs every gate end-to-end; all
pass. Rev-1 board audited retroactively: Q1 was the only netless part.

Co-Authored-By: Claude Fable 5 <noreply@anthropic.com>
Routing:
- net FLOAT1_SW: track 88.1 -> 138.8 mm, vias 2 -> 1
- net CH1_OUT: track 116.2 -> 76.5 mm, vias 0 -> 1
- net +5V_BUCK: track 58.7 -> 95.6 mm, vias 3 -> 2
- net CH3_OUT: track 54.3 -> 90.0 mm
- net FLOAT2_SW: track 92.2 -> 125.1 mm
- net GND: track 290.9 -> 313.5 mm, vias 1 -> 0
- net RLY3_DRV: track 56.6 -> 75.2 mm
- net +3V3: track 175.2 -> 157.2 mm
- net +12V: track 189.4 -> 174.9 mm, vias 2 -> 3
- net RLY2_DRV: track 96.9 -> 86.7 mm
- net +12V_F: track 68.7 -> 78.2 mm
- net LED1_A: track 62.1 -> 71.2 mm, vias 3 -> 1
- net FLOAT1_GPIO: track 39.5 -> 48.3 mm
- net +5V: track 74.5 -> 67.2 mm
- net RLY1_DRV: track 50.0 -> 44.4 mm
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
Commit message: HAT rev 2: production-ready 5V link, visible title, deterministic routing
- JP1 hand-soldered jumper replaced by machine-placed 0R (R21): boards
  leave assembly fully powered, no per-board hand step for inventory;
  remove with an iron to isolate the buck for debug.
- 'ExoPet HAT rev2' title moved from under the relays to the top-edge
  strip where it stays visible assembled.
- Route pipeline de-lotteried: DSN exports with the board edge inset
  0.2mm in memory (kills copper-to-edge shaves) and the locked +3V3
  pre-route extends through the EEPROM cluster (C4->R3->R4), which the
  router stranded on varying seeds. Preflight fully green: DRC 0/0,
  golden 208-pin audit, fab cross-check (62 refs). Mockups refreshed.

Co-Authored-By: Claude Fable 5 <noreply@anthropic.com>
Parts:
- removed JP1: SolderJumper-2_P1.3mm_Open_RoundedPad1.0x1.5mm, Jumper:SolderJumper-2_P1.3mm_Open_RoundedPad1.0x1.5mm
- added R21: R_0805_2012Metric, Resistor_SMD:R_0805_2012Metric, B.Cu at (14.8, 46.0)
Routing:
- net FLOAT1_SW: track 138.8 -> 88.5 mm, vias 1 -> 2
- net FLOAT2_SW: track 125.1 -> 81.9 mm
- net CH3_OUT: track 90.0 -> 52.3 mm
- net +5V_BUCK: track 95.6 -> 59.2 mm, vias 2 -> 3
- net GND: track 313.5 -> 287.9 mm, vias 0 -> 3
- net +3V3: track 157.2 -> 179.8 mm, vias 2 -> 3
- net RLY3_DRV: track 75.2 -> 55.2 mm
- net RLY4_DRV: track 69.1 -> 89.0 mm, vias 1 -> 0
- net LED3_A: track 35.1 -> 53.5 mm
- net LED1_A: track 71.2 -> 55.7 mm
- net RLY2_DRV: track 86.7 -> 72.3 mm
- net +5V: track 67.2 -> 81.5 mm
- net CH1_FUSED: track 31.6 -> 43.6 mm
- net CH1_OUT: track 76.5 -> 88.4 mm, vias 1 -> 2
- net GPIO17: track 47.4 -> 57.9 mm
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
Commit message: HAT rev 2 + enclosure: DS18B20 R/Y/B wire markings; R21 current-rating fix; hard-fail preflight
'Are you sure' audit of my own R21 change found three real issues:
C17477 was an unverified from-memory LCSC code; an 0805 zero-ohm
jumper (~2A) under-rates the Pi 4's 3A-peak 5V rail; and preflight's
piped exit codes meant gates could not actually fail the run. R21 is
now a 1206 with a rated>=3A matching hint, relocated collision-free,
and preflight hard-fails on any gate via explicit pass-token checks.

TEMP terminal gets R/Y/B markings (DS18B20 red=3V3, yellow=data,
black=GND) on both the board silk and the enclosure lid beside the
screw slot. All gates green.

Co-Authored-By: Claude Fable 5 <noreply@anthropic.com>
Parts:
- R21: value R_0805_2012Metric -> R_1206_3216Metric; footprint Resistor_SMD:R_0805_2012Metric -> Resistor_SMD:R_1206_3216Metric
- moved R21 3.01 mm to (14.0, 48.9)
Routing:
- net CH2_OUT: track 72.3 -> 113.0 mm
- net FLOAT2_GPIO: track 56.4 -> 83.5 mm
- net GND: track 287.9 -> 309.2 mm, vias 3 -> 1
- net RLY4_DRV: track 89.0 -> 71.9 mm, vias 0 -> 1
- net FLOAT2_SW: track 81.9 -> 97.5 mm
- net +5V: track 81.5 -> 66.1 mm
- net CH1_FUSED: track 43.6 -> 29.6 mm
- net LED3_A: track 53.5 -> 42.9 mm
- net LED1_A: track 55.7 -> 65.4 mm
- net +5V_BUCK: track 59.2 -> 68.5 mm
- net GPIO17: track 57.9 -> 48.7 mm
- net GPIO27: track 47.4 -> 54.7 mm
- net CH3_FUSED: track 33.8 -> 27.0 mm, vias 1 -> 0
- net CH2_FUSED: track 44.6 -> 38.2 mm
- net LED4_A: track 36.1 -> 30.8 mm
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Other:
- board text added: "B"
- board text added: "R"
- board text added: "Y"
