File: hardware/exopet-hat/exopet-hat.kicad_sch (KiCad schematic)
At the start: 69 parts, among them J1 12V DC in, J10 CH3 12V OUT, J11 CH4 dry contact, J13 FLOAT1 switch, J14 FLOAT2 switch, J3 RPi GPIO (HAT), J4 TEMP (3V3/DATA/GND), J8 CH1 12V OUT, J9 CH2 12V OUT, K1 G5LE-1-CF DC12, K2 G5LE-1-CF DC12, K3 G5LE-1-CF DC12, K4 G5LE-1-CF DC12, Q1 AOD403, U2 TBD62003AFG, U4 CAT24C32, U5 5V ESD clamp (SOD-323), U6 TPS54302DDC

Commit message: HAT rev 3: schematic — isolated pH subsystem + supervised float ADC
New components: ADS1115 x2 (floats 0x48 main / pH 0x49 isolated),
ISO1540 I2C isolator, MCP6002 pH buffers (probe follower + buffered
mid-rail reference driving the BNC shield), B0505S-class isolated
DC-DC (custom SIP-4 footprint, local ExoPet.pretty lib), edge-launch
BNC, bias/pullup/decoupling passives, 10k float-sense taps. J3 pins
3/5 become I2C1. Generator gains 'extends' resolution (derived
symbols like ADS1115IDGS/MCP6002 carry no pins of their own) and
multi-unit emission (op-amp A/B/power units all instantiated — ERC
caught unit 2/3 pins dangling out of the netlist, a Q1-class miss).
Netlist verified pin-by-pin; polarity lint clean; ERC benign-only.

Co-Authored-By: Claude Fable 5 <noreply@anthropic.com>
Parts:
- added C18, C20, C21, C25: 100nF, Capacitor_SMD:C_0805_2012Metric, symbol Device:C
- added C22: 10uF 10V, Capacitor_SMD:C_1206_3216Metric, symbol Device:C
- added C26: 100nF (bias), Capacitor_SMD:C_0805_2012Metric, symbol Device:C
- added C27: 4.7uF 25V, Capacitor_SMD:C_1206_3216Metric, symbol Device:C
- added J15: pH probe BNC, Connector_Coaxial:BNC_Amphenol_031-6575_Horizontal, symbol Connector:Conn_Coaxial
- added PS1: B0505S-1WR2 iso DC-DC (SIP-4), ExoPet:Converter_DCDC_B0505S-1W_SIP4, symbol Connector_Generic:Conn_01x04
- added R22, R23: 10k, Resistor_SMD:R_0805_2012Metric, symbol Device:R
- added R24: 100k (bias hi), Resistor_SMD:R_0805_2012Metric, symbol Device:R
- added R25: 100k (bias lo), Resistor_SMD:R_0805_2012Metric, symbol Device:R
- added R26: 4.7k (iso SDA pullup), Resistor_SMD:R_0805_2012Metric, symbol Device:R
- added R27: 4.7k (iso SCL pullup), Resistor_SMD:R_0805_2012Metric, symbol Device:R
- added U10: MCP6002 (pH buffers), Package_SO:SOIC-8_3.9x4.9mm_P1.27mm, symbol Amplifier_Operational:MCP6002-xSN
- added U7: ADS1115 (floats, 0x48), Package_SO:MSOP-10_3x3mm_P0.5mm, symbol Analog_ADC:ADS1115IDGS
- added U8: ADS1115 (pH, 0x49), Package_SO:MSOP-10_3x3mm_P0.5mm, symbol Analog_ADC:ADS1115IDGS
- added U9: ISO1540 I2C isolator, Package_SO:SOIC-8_3.9x4.9mm_P1.27mm, symbol Isolator:ISO1540
Connections:
- net +3V3: now also C18.1, C20.1, U7.8 (VDD), U9.1 (VCC1)
- net +5V_BUCK: now also C27.1, PS1.1 (Pin_1)
- net FLOAT1_SW: now also R22.1
- net FLOAT2_SW: now also R23.1
- net GND: now also C18.2, C20.2, C27.2, PS1.2 (Pin_2), U7.1 (ADDR), U7.3 (GND), U7.6 (AIN2), U7.7 (AIN3), U9.4 (GND1)
- net I2C1_SDA: now reaches J3.3 (SDA/GPIO2)
- net I2C1_SDA: now also U7.9 (SDA), U9.2 (SDA1)
- net I2C1_SCL: now reaches J3.5 (SCL/GPIO3)
- net I2C1_SCL: now also U7.10 (SCL), U9.3 (SCL1)
- new net +5V_ISO: C21.1, C22.1, C25.1, PS1.4 (Pin_4), R24.1, R26.1, R27.1, U10.8 (V+), U8.1 (ADDR), U8.8 (VDD), U9.8 (VCC2)
- new net BIAS_MID: C26.1, R24.2, R25.1, U10.5 (+)
- new net FLT1_SENSE: R22.2, U7.4 (AIN0)
- new net FLT2_SENSE: R23.2, U7.5 (AIN1)
- new net ISO_GND: C21.2, C22.2, C25.2, C26.2, PS1.3 (Pin_3), R25.2, U10.4 (V-), U8.3 (GND), U8.6 (AIN2), U8.7 (AIN3), U9.5 (GND2)
- new net ISO_SCL: R27.2, U8.10 (SCL), U9.6 (SCL2)
- new net ISO_SDA: R26.2, U8.9 (SDA), U9.7 (SDA2)
- new net PH_BUF: U10.1, U10.2 (-), U8.4 (AIN0)
- new net PH_IN: J15.1 (In), U10.3 (+)
- new net PH_REF: J15.2 (Ext), U10.6 (-), U10.7, U8.5 (AIN1)
